File: kicad/EtherKraken.kicad_pcb (KiCad board)
At the start: 2 copper layers, 87.6 x 100.8 mm, 56 parts, among them IC1 NCV33375ST3.3T3G, IC2 NCV33375ST3.3T3G, J1 Conn_02x03_Odd_Even, J2 Conn_02x10_Odd_Even, J3 RJ45_Wuerth_7499010121A, J4 Conn_02x10_Odd_Even, J5 Conn_02x10_Odd_Even, U1 RASPBERRY_PI_ZERO_2_W, U2 AT45DB641E-SHN-T, U3 W5500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

Commit message: Implement basic board initialization and flash interface in HAL
Parts:
- RN1: footprint parts:R_Array_Convex_8N_1206 -> Resistor_SMD:R_Array_Convex_4x1206
Connections:
- net EXT_CTRL0 renamed CTRL2
- net EXT_CTRL1 renamed CTRL1
- net EXT_INT renamed CTRL0
- net EXT_IO_RST renamed CTRL5
- net EXT_OLED_DC renamed CTRL4
- net EXT_OLED_RST renamed CTRL3
