File: kicad/EtherKraken.kicad_pcb (KiCad board)
At the start: 2 copper layers, 87.6 x 100.8 mm, 56 parts, among them IC1 NCV33375ST3.3T3G, IC2 NCV33375ST3.3T3G, J1 Conn_02x03_Odd_Even, J2 Conn_02x10_Odd_Even, J3 RJ45_Wuerth_7499010121A, J4 Conn_02x10_Odd_Even, J5 Conn_02x10_Odd_Even, U1 RASPBERRY_PI_ZERO_2_W, U2 AT45DB641E-SHN-T, U3 W5500, U4 MCP23017x-x-SO, U5 MCP23017x-x-SO, Y1 25MHz

Commit message: Update KiCad files for Revision B
Parts:
- removed the J4 at (122.2, 74.8)
- removed the R2 at (51.0, 91.4)
- added C22: 18pF, Capacitor_SMD:C_1206_3216Metric, F.Cu at (100.7, 90.5)
- added C23: 100nF, Capacitor_SMD:C_1206_3216Metric, F.Cu at (81.7, 87.5)
- added C24: 100nF, Capacitor_SMD:C_1206_3216Metric, F.Cu at (92.4, 99.8)
- added C25: 100nF, Capacitor_SMD:C_1206_3216Metric, F.Cu at (90.1, 101.5)
- added C26: 100nF, Capacitor_SMD:C_1206_3216Metric, F.Cu at (91.9, 88.4)
- added C27: 100nF, Capacitor_SMD:C_1206_3216Metric, F.Cu at (81.7, 100.1)
- added C28: 22pF, Capacitor_SMD:C_1206_3216Metric, F.Cu at (111.0, 103.3)
- added C29: 33pF, Capacitor_SMD:C_1206_3216Metric, F.Cu at (111.0, 98.4)
- added C30: 100nF, Capacitor_SMD:C_1206_3216Metric, F.Cu at (101.6, 99.3)
- added D4: LED, LED_SMD:LED_1206_3216Metric, F.Cu at (112.2, 91.5)
- added D5: LED, LED_SMD:LED_1206_3216Metric, F.Cu at (112.2, 89.0)
- added D6: LED, LED_SMD:LED_1206_3216Metric, F.Cu at (112.2, 86.5)
- added D7: LED, LED_SMD:LED_1206_3216Metric, F.Cu at (112.2, 84.0)
- added J3: Conn_02x10_Odd_Even, parts:09185206324_02x10_P2.54, F.Cu at (122.1, 74.5)
- added Q1: MMBT3904, Package_TO_SOT_SMD:SOT-23, F.Cu at (87.4, 58.0)
- added Q2: MMBT3904, Package_TO_SOT_SMD:SOT-23, F.Cu at (87.4, 61.5)
- added Q3: MMBT3904, Package_TO_SOT_SMD:SOT-23, F.Cu at (87.4, 65.1)
- added Q4: MMBT3904, Package_TO_SOT_SMD:SOT-23, F.Cu at (87.4, 68.6)
- added R14: 1,2k, Resistor_SMD:R_1206_3216Metric, F.Cu at (93.2, 57.6)
- added R15: 62R, Resistor_SMD:R_1206_3216Metric, F.Cu at (91.2, 79.6)
- added R16: 1,2k, Resistor_SMD:R_1206_3216Metric, F.Cu at (93.2, 60.1)
- added R17: 62R, Resistor_SMD:R_1206_3216Metric, F.Cu at (91.2, 77.1)
- added R18: 1,2k, Resistor_SMD:R_1206_3216Metric, F.Cu at (93.2, 62.6)
- added R19: 62R, Resistor_SMD:R_1206_3216Metric, F.Cu at (91.2, 74.6)
- added R20: 1,2k, Resistor_SMD:R_1206_3216Metric, F.Cu at (93.2, 65.1)
- added R21: 62R, Resistor_SMD:R_1206_3216Metric, F.Cu at (91.2, 72.1)
- added R22: 10k, Resistor_SMD:R_1206_3216Metric, F.Cu at (92.4, 106.3)
- added U6: SC16IS740, Package_SO:TSSOP-16_4.4x5mm_P0.65mm, F.Cu at (98.6, 103.5)
- added Y2: 8MHz, Crystal:Crystal_HC49-U_Vertical, F.Cu at (96.4, 96.8)
- added Y3: 1,8432MHz, Crystal:Crystal_HC49-U_Vertical, F.Cu at (106.9, 104.8)
- C20: moved to F.Cu
- C21: value 100nF -> 18pF; moved to F.Cu
- D1, D2, D3: footprint LED_THT:LED_D3.0mm -> LED_SMD:LED_1206_3216Metric
- RN1: value 3,3R -> 33R; footprint Resistor_SMD:R_Array_Convex_4x1206 -> parts:R_Array_Convex_8N_1206
- U5: value MCP23017x-x-SO -> STM32F071CBTx; footprint Package_SO:SOIC-28W_7.5x17.9mm_P1.27mm -> Package_QFP:LQFP-48_7x7mm_P0.5mm
- moved C20 29.6 mm to (94.0, 68.0), turned to 0 degrees
- moved C21 18.5 mm to (100.7, 95.3)
- moved U4 11.2 mm to (103.0, 66.0)
- moved U5 7.83 mm to (86.2, 93.9), turned to 180 degrees
- moved C4 2.10 mm to (48.1, 90.0)
- moved D3 1.76 mm to (105.5, 135.6), turned to -90 degrees
- moved D2 1.36 mm to (91.6, 111.8)
- moved D1 1.29 mm to (80.8, 111.8)
- moved R12 0.28 mm to (95.2, 112.0)
- moved R11 0.28 mm to (84.4, 112.0)
- moved J5 0.15 mm to (122.1, 110.8)
- renumbered C11 to C10, C10 to C11, J3 to J4, R11 to R10, R12 to R11, R13 to R12, R14 to R13, R3 to R2, R4 to R3, R5 to R4, R6 to R5, R7 to R6, R8 to R7, R9 to R8, R10 to R9
Connections:
- net CTRL2 renamed CO_SINT
- C21 pad 1: GND -> Net-(U5-PF0)
- C21 pad 2: VCC3.3 -> GND
- J2 pad 10: CTRL1 -> CO_BOOT
- J2 pad 14: CTRL3 -> AUX0
- J2 pad 16: CTRL4 -> AUX1
- J2 pad 18: CTRL5 -> AUX_PWR_EN
- J2 pad 7: SPI1_CE0 -> GND
- J2 pad 8: CTRL0 -> CO_RST
- J5 pad 10: Net-(J5-Pin_10) -> IO_B9
- J5 pad 11: Net-(J5-Pin_11) -> IO_A14
- J5 pad 12: Net-(J5-Pin_12) -> IO_B10
- J5 pad 13: Net-(J5-Pin_13) -> IO_A15
- J5 pad 14: Net-(J5-Pin_14) -> IO_B11
- J5 pad 15: Net-(J5-Pin_15) -> IO_A16
- J5 pad 16: Net-(J5-Pin_16) -> IO_A18
- J5 pad 17: Net-(J5-Pin_17) -> IO_A17
- J5 pad 18: Net-(J5-Pin_18) -> IO_A19
- J5 pad 3: Net-(J5-Pin_3) -> IO_A10
- J5 pad 4: Net-(J5-Pin_4) -> IO_B6
- J5 pad 5: Net-(J5-Pin_5) -> IO_A11
- J5 pad 6: Net-(J5-Pin_6) -> IO_B7
- J5 pad 7: Net-(J5-Pin_7) -> IO_A12
- J5 pad 8: Net-(J5-Pin_8) -> IO_B8
- J5 pad 9: Net-(J5-Pin_9) -> IO_A13
- U1 pad 15: CTRL4 -> CO_RST
- U1 pad 16: CTRL3 -> CO_BOOT
- U1 pad 22: CTRL1 -> AUX0
- U1 pad 29: IO_RST0 -> IO_INT1
- U1 pad 31: IO_RST1 -> IO_RST
- U1 pad 33: CTRL0 -> ETH_RST
- U1 pad 37: CTRL5 -> AUX1
- U1 pad 7: ETH_RST -> IO_INT0
- U2 pad 5: Net-(U2-~{WP}) -> VCC3.3
- U4 pad 1: Net-(J4-Pin_4) -> IO_B8
- U4 pad 18: IO_RST0 -> IO_RST
- U4 pad 19: unconnected-(U4-INTB-Pad19) -> IO_INT1
- U4 pad 2: Net-(J4-Pin_6) -> IO_B9
- U4 pad 20: unconnected-(U4-INTA-Pad20) -> IO_INT0
- U4 pad 21: Net-(J4-Pin_3) -> IO_B0
- U4 pad 22: Net-(J4-Pin_5) -> IO_B1
- U4 pad 23: Net-(J4-Pin_7) -> IO_B2
- U4 pad 24: Net-(J4-Pin_9) -> IO_B3
- U4 pad 25: Net-(J4-Pin_11) -> IO_B4
- U4 pad 26: Net-(J4-Pin_13) -> IO_B5
- U4 pad 27: Net-(J4-Pin_15) -> IO_B6
- U4 pad 28: Net-(J4-Pin_17) -> IO_B7
- U4 pad 3: Net-(J4-Pin_8) -> IO_B10
- U4 pad 4: Net-(J4-Pin_10) -> IO_B11
- U4 pad 5: Net-(J4-Pin_12) -> ST_LED0
- U4 pad 6: Net-(J4-Pin_14) -> ST_LED1
- U4 pad 7: Net-(J4-Pin_16) -> ST_LED2
- U4 pad 8: Net-(J4-Pin_18) -> ST_LED3
- U5 pad 1: Net-(J5-Pin_4) -> VCC3.3
- U5 pad 10: GND -> IO_A0
- U5 pad 11: unconnected-(U5-NC-Pad11) -> IO_A1
- U5 pad 12: I2C_SCL -> IO_A2
- U5 pad 13: I2C_SDA -> IO_A3
- U5 pad 14: unconnected-(U5-NC-Pad14) -> IO_A4
- U5 pad 15: VCC3.3 -> IO_A5
- U5 pad 16: GND -> IO_A6
- U5 pad 17: GND -> IO_A7
- U5 pad 18: IO_RST1 -> IO_A9
- U5 pad 19: unconnected-(U5-INTB-Pad19) -> IO_A10
- U5 pad 2: Net-(J5-Pin_6) -> unconnected-(U5-PC13-Pad2)
- U5 pad 20: unconnected-(U5-INTA-Pad20) -> IO_A11
- U5 pad 21: Net-(J5-Pin_3) -> unconnected-(U5-PB10-Pad21)
- U5 pad 22: Net-(J5-Pin_5) -> unconnected-(U5-PB11-Pad22)
- U5 pad 23: Net-(J5-Pin_7) -> GND
- U5 pad 24: Net-(J5-Pin_9) -> VCC3.3
- U5 pad 25: Net-(J5-Pin_11) -> SPI1_CE0
- U5 pad 26: Net-(J5-Pin_13) -> SPI1_SCLK
- U5 pad 27: Net-(J5-Pin_15) -> SPI1_MISO
- U5 pad 28: Net-(J5-Pin_17) -> SPI1_MOSI
- U5 pad 3: Net-(J5-Pin_8) -> unconnected-(U5-PC14-Pad3)
- U5 pad 4: Net-(J5-Pin_10) -> unconnected-(U5-PC15-Pad4)
- U5 pad 5: Net-(J5-Pin_12) -> Net-(U5-PF0)
- U5 pad 6: Net-(J5-Pin_14) -> Net-(U5-PF1)
- U5 pad 7: Net-(J5-Pin_16) -> CO_RST
- U5 pad 8: Net-(J5-Pin_18) -> GND
Routing:
- net CO_BOOT: track 0.00 -> 88.1 mm, vias 0 -> 5
- net IO_A17: track 0.00 -> 86.0 mm, vias 0 -> 10
- net IO_A19: track 0.00 -> 81.8 mm, vias 0 -> 10
- net IO_A18: track 0.00 -> 80.6 mm, vias 0 -> 10
- net CO_RST: track 0.00 -> 80.2 mm, vias 0 -> 6
- net IO_RST0: track 78.5 -> 0.00 mm
- net CO_SINT: track 45.7 -> 123.1 mm, vias 2 -> 6
- net CTRL0: track 75.3 -> 0.00 mm, vias 2 -> 0
- net IO_A8: track 0.00 -> 71.9 mm, vias 0 -> 5
- net AUX1: track 0.00 -> 68.9 mm, vias 0 -> 2
- net AUX0: track 0.00 -> 68.7 mm, vias 0 -> 2
- net IO_RST1: track 67.4 -> 0.00 mm
- net Net-(J5-Pin_4): track 66.2 -> 0.00 mm, vias 1 -> 0
- net CTRL5: track 65.2 -> 0.00 mm, vias 2 -> 0
- net IO_INT0: track 0.00 -> 65.1 mm, vias 0 -> 2
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- added copper zone on B.Cu, net VCC3.3
- added copper zone on F.Cu, net VCC3.3
- added copper zone on F.Cu, net VCC3.3A
Other:
- board text added: "AUX PWR"
- board text added: "COPROCESSOR"
- board text added: "ETHERNET"
- board text added: "EtherKraken"
- board text added: "GPIO"
- board text added: "STATUS"
- board text removed: "CE0"
- board text removed: "CE1"
- board text removed: "CE2"
- board text removed: "CTR0"
- board text removed: "CTR1"
- board text removed: "CTR2"
- board text removed: "CTR3"
- board text removed: "CTR4"
- board text removed: "CTR5"
- board text removed: "EtherKraken V1 Revision B"
- board text removed: "IO0"
- board text removed: "IO10"
- board text removed: "IO11"
- board text removed: "IO12"
- board text removed: "IO13"
- board text removed: "IO14"
- board text removed: "IO15"
- board text removed: "IO3"
- board text removed: "IO4"
- board text removed: "IO5"
- board text removed: "IO6"
- board text removed: "IO7"
- board text removed: "IO8"
- board text removed: "IO9"
- board text removed: "I²C:0x20"
- board text removed: "I²C:0x21"
- board text removed: "MISO"
- board text removed: "MOSI"
- board text removed: "RX"
- board text removed: "SCL"
- board text removed: "SCLK"
- board text removed: "SDA"
- board text removed: "TX"
