File: kicad/EtherKraken.kicad_pcb (KiCad board)
At the start: 2 copper layers, 87.6 x 100.8 mm, 84 parts, among them IC1 NCV33375ST3.3T3G, IC2 NCV33375ST3.3T3G, J1 Conn_02x03_Odd_Even, J2 Conn_02x10_Odd_Even, J3 Conn_02x10_Odd_Even, J4 RJ45_Wuerth_7499010121A, J5 Conn_02x10_Odd_Even, Q1 MMBT3904, Q2 MMBT3904, Q3 MMBT3904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

Commit message: Split single A2 sheet for schematic into multiple A4 sub schematics
Parts:
- removed C1: 2,2µF, Capacitor_THT:CP_Radial_D5.0mm_P2.00mm
- removed C10, C12, C14, C17, C2, C20, C23, C24, C25, C26, C27, C30, C4, C6: 100nF, Capacitor_SMD:C_1206_3216Metric
- removed C11, C3: 4,7µF, Capacitor_THT:CP_Radial_D5.0mm_P2.00mm
- removed C13, C5: 10µF, Capacitor_THT:CP_Radial_D5.0mm_P2.00mm
- removed C15, C16: 6.8nF, Capacitor_SMD:C_1206_3216Metric
- removed C18: 10nF, Capacitor_SMD:C_1206_3216Metric
- removed C19: 4.7µF, Capacitor_THT:CP_Radial_D5.0mm_P2.00mm
- removed C21, C22, C7, C8: 18pF, Capacitor_SMD:C_1206_3216Metric
- removed C28: 22pF, Capacitor_SMD:C_1206_3216Metric
- removed C29: 33pF, Capacitor_SMD:C_1206_3216Metric
- removed C9: 22nF, Capacitor_SMD:C_1206_3216Metric
- removed D1, D2, D3, D4, D5, D6, D7: LED, LED_SMD:LED_1206_3216Metric
- removed H1, H2, H3, H4: M3, MountingHole:MountingHole_3.2mm_M3_DIN965_Pad
- removed IC1, IC2: NCV33375ST3.3T3G, parts:SOT230P700X175-4N
- removed J1: Conn_02x03_Odd_Even, parts:09185066324_02x03_P2.54
- removed J2, J3, J5: Conn_02x10_Odd_Even, parts:09185206324_02x10_P2.54
- removed J4: RJ45_Wuerth_7499010121A, Connector_RJ:RJ45_Wuerth_7499010121A_Horizontal
- removed Q1, Q2, Q3, Q4: MMBT3904, Package_TO_SOT_SMD:SOT-23
- removed R1, R22: 10k, Resistor_SMD:R_1206_3216Metric
- removed R10: 12.4k, Resistor_SMD:R_1206_3216Metric
- removed R11, R12: 51R, Resistor_SMD:R_1206_3216Metric
- removed R13: 150R, Resistor_SMD:R_1206_3216Metric
- removed R14, R16, R18, R20: 1,2k, Resistor_SMD:R_1206_3216Metric
- removed R15, R17, R19, R21: 62R, Resistor_SMD:R_1206_3216Metric
- removed R2: 1M, Resistor_SMD:R_1206_3216Metric
- removed R3, R4, R6, R7: 49,9R, Resistor_SMD:R_1206_3216Metric
- removed R5: 10R, Resistor_SMD:R_1206_3216Metric
- removed R8, R9: 330R, Resistor_SMD:R_1206_3216Metric
- removed RN1: 33R, parts:R_Array_Convex_8N_1206
- removed U1: RASPBERRY_PI_ZERO_2_W, parts:MODULE_RASPBERRY_PI_ZERO_2_W
- removed U2: AT45DB641E-SHN-T, Package_SO:SOIC-8_5.3x5.3mm_P1.27mm
- removed U3: W5500, Package_QFP:LQFP-48_7x7mm_P0.5mm
- removed U4: MCP23017x-x-SO, Package_SO:SOIC-28W_7.5x17.9mm_P1.27mm
- removed U5: STM32F071CBTx, Package_QFP:LQFP-48_7x7mm_P0.5mm
- removed U6: SC16IS740, Package_SO:TSSOP-16_4.4x5mm_P0.65mm
- removed Y1: 25MHz, Crystal:Crystal_HC49-U_Vertical
- removed Y2: 8MHz, Crystal:Crystal_HC49-U_Vertical
- removed Y3: 1,8432MHz, Crystal:Crystal_HC49-U_Vertical
Routing:
- net VCC5: track 275.2 -> 0.00 mm, vias 1 -> 0
- net VCC3.3: track 175.6 -> 0.00 mm, vias 4 -> 0
- net AUX_PWR_EN: track 150.2 -> 0.00 mm, vias 7 -> 0
- net CO_SINT: track 123.1 -> 0.00 mm, vias 6 -> 0
- net I2C_SCL: track 121.7 -> 0.00 mm, vias 5 -> 0
- net I2C_SDA: track 118.1 -> 0.00 mm, vias 5 -> 0
- net SPI0_MOSI: track 109.7 -> 0.00 mm, vias 3 -> 0
- net SPI0_MISO: track 104.9 -> 0.00 mm, vias 3 -> 0
- net SPI0_SCLK: track 103.7 -> 0.00 mm, vias 5 -> 0
- net SPI1_SCLK: track 90.7 -> 0.00 mm, vias 3 -> 0
- net ETH_RST: track 89.6 -> 0.00 mm, vias 2 -> 0
- net SPI0_CE0: track 88.2 -> 0.00 mm, vias 3 -> 0
- net ETH_INT: track 88.1 -> 0.00 mm, vias 3 -> 0
- net CO_BOOT: track 88.1 -> 0.00 mm, vias 5 -> 0
- net SPI1_MOSI: track 87.2 -> 0.00 mm, vias 4 -> 0
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- removed copper zone on B.Cu, net Earth_Clean
- removed copper zone on F.Cu, net Earth_Clean
- removed copper zone on B.Cu, net GND
- removed copper zone on F.Cu, net GND
- removed copper zone on B.Cu, net VCC3.3
- removed copper zone on F.Cu, net VCC3.3
- removed copper zone on F.Cu, net VCC3.3A
Other:
- board outline removed
- board text removed: "3.3V(A)"
- board text removed: "3.3V(D)"
- board text removed: "5V"
- board text removed: "AUX PWR"
- board text removed: "COPROCESSOR"
- board text removed: "ETH"
- board text removed: "ETHERNET"
- board text removed: "EXT"
- board text removed: "EtherKraken"
- board text removed: "GND"
- board text removed: "GPIO"
- board text removed: "IO1"
- board text removed: "IO2"
- board text removed: "Karma Krafts"
- board text removed: "Made in Germany"
- board text removed: "PN:01011B"
- board text removed: "PWR"
- board text removed: "SN:032601"
- board text removed: "STATUS"
