File: kicad/Coprocessor.kicad_sch (KiCad schematic)
At the start: 12 parts, among them U10 STM32F071CBTx, Y3 8MHz

Commit message: Add main bus to root schematic, use bus labels for exporting IO and CPIO busses
Connections:
- net A0 renamed CPIO0
- net A1 renamed CPIO1
- net A10 renamed CPIO10
- net A11 renamed CPIO11
- net A12 renamed CPIO12
- net A13 renamed CPIO13
- net A14 renamed CPIO14
- net A15 renamed CPIO15
- net A16 renamed CPIO16
- net A17 renamed CPIO17
- net A18 renamed CPIO18
- net A19 renamed CPIO19
- net A2 renamed CPIO2
- net A3 renamed CPIO3
- net A4 renamed CPIO4
- net A5 renamed CPIO5
- net A6 renamed CPIO6
- net A7 renamed CPIO7
- net A8 renamed CPIO8
- net A9 renamed CPIO9
- net CO_BOOT renamed BOOT
- net CO_RST renamed RST
- net CO_SCTS renamed CTS
- net CO_SRTS renamed RTS
- net CO_SRX renamed RX
- net CO_STX renamed TX
- net CO_ST_LED0 renamed CPIO20
- net CO_ST_LED1 renamed CPIO21
- net CO_ST_LED2 renamed CPIO22
- net CO_ST_LED3 renamed CPIO23
- net SPI1_CE0 renamed CS
- net SPI1_MISO renamed MISO
- net SPI1_MOSI renamed MOSI
- net SPI1_SCLK renamed SCLK
