File: kicad/Fan Controller.kicad_sch (KiCad schematic)
At the start: 11 parts, among them M1 Fan_4pin, M2 Fan_4pin, Q1 MMBT2222A, Q2 MMBT2222A, U11 EMC2302-x-AIZL

Commit message: Add main bus to root schematic, use bus labels for exporting IO and CPIO busses
Connections:
- net I2C_SCL renamed SCL
- net I2C_SDA renamed SDA
Changed lines of the file:
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@@
 		(at 106.68 88.9)
 	)
-	(bus_entry
-		(at 62.23 78.74)
-		(size 2.54 2.54)
-		(stroke
-			(width 0)
-			(type default)
-		)
-	)
-	(bus_entry
-		(at 62.23 81.28)
-		(size 2.54 2.54)
-		(stroke
-			(width 0)
-			(type default)
-		)
-	)
 	(wire
 		(pts
@@
 	(wire
 		(pts
+			(xy 57.15 83.82) (xy 106.68 83.82)
+		)
+		(stroke
+			(width 0)
+			(type default)
+		)
+	)
+	(wire
+		(pts
 			(xy 185.42 82.55) (xy 186.69 82.55)
 		)
@@
 	(wire
 		(pts
-			(xy 64.77 81.28) (xy 106.68 81.28)
-		)
-		(stroke
-			(width 0)
-			(type default)
-		)
-	)
-	(wire
-		(pts
 			(xy 199.39 90.17) (xy 199.39 87.63)
 		)
@@
 		)
 	)
-	(bus
-		(pts
-			(xy 55.88 76.2) (xy 62.23 76.2)
+	(wire
+		(pts
+			(xy 57.15 81.28) (xy 106.68 81.28)
 		)
 		(stroke
@@
 		)
 	)
-	(bus
-		(pts
-			(xy 62.23 76.2) (xy 62.23 81.28)
-		)
-		(stroke
-			(width 0)
-			(type default)
-		)
-	)
 	(wire
 		(pts
@@
 		(pts
 			(xy 166.37 69.85) (xy 166.37 97.79)
-		)
-		(stroke
-			(width 0)
-			(type default)
-		)
-	)
-	(wire
-		(pts
-			(xy 64.77 83.82) (xy 106.68 83.82)
 		)
 		(stroke
@@
 		)
 	)
-	(hierarchical_label "MP"
-		(shape bidirectional)
-		(at 55.88 76.2 180)
+	(hierarchical_label "SCL"
+		(shape input)
+		(at 57.15 83.82 180)
 		(effects
 			(font
@@
 		(effects
 			(font
+				(size 1.27 1.27)
+			)
+			(justify right)
+		)
+	)
+	(hierarchical_label "SDA"
+		(shape bidirectional)
+		(at 57.15 81.28 180)
+		(effects
+			(font
