File: kicad/Main Processor.kicad_sch (KiCad schematic)
At the start: 15 parts, among them U6 RASPBERRY_PI_ZERO_2_W, U7 AT45DB641E-SHN-T, U8 MCP23017x-x-SO, U9 SC16IS740, Y2 1,8432MHz

Commit message: Add main bus to root schematic, use bus labels for exporting IO and CPIO busses
Connections:
- net B0 renamed IO0
- net B1 renamed IO1
- net B10 renamed IO10
- net B11 renamed IO11
- net B12 renamed IO12
- net B13 renamed IO13
- net B14 renamed IO14
- net B15 renamed IO15
- net B2 renamed IO2
- net B3 renamed IO3
- net B4 renamed IO4
- net B5 renamed IO5
- net B6 renamed IO6
- net B7 renamed IO7
- net B8 renamed IO8
- net B9 renamed IO9
Other:
- note added: "RX/TX pairs need to be flipped"
- moved on the sheet: C24, C25, C26, C27, C28, C29, C30, R15, RN4, RN5, U6, U7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
