File: kicad/Ethernet PHY.kicad_sch (KiCad schematic)
At the start: 32 parts, among them J2 RJ45_Wuerth_7499010121A, U5 W5500, Y1 25MHz

Commit message: Add main bus to root schematic, use bus labels for exporting IO and CPIO busses
Connections:
- net ETH_INT renamed INT
- net ETH_RST renamed RST
- net SPI0_CS0 renamed CS
- net SPI0_MISO renamed MISO
- net SPI0_MOSI renamed MOSI
- net SPI0_SCLK renamed SCLK
Other:
- moved on the sheet: C10, C11, C12, C13, C14, C15, C16, C17, C18, C19, C20, C21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

Commit message: Add EtherKraken V1 Rev. C schematics as PDF to docs
Other:
- note added: "Clean earth should be connected to the digital ground (GND) through a 1nF/Y2 capacitor to create a clean star grounding path for EMI"
- note removed: "Clean earth should be connected to the chassis through a 1nF/Y2 capacitor to create a clean star grounding path for EMI"
Changed lines of the file:
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@@
 		)
 	)
-	(text "Clean earth should be connected to the \nchassis through a 1nF/Y2 capacitor to \ncreate a clean star grounding path for EMI"
+	(text "Clean earth should be connected to the \ndigital ground (GND) through a 1nF/Y2 capacitor to \ncreate a clean star grounding path for EMI"
 		(exclude_from_sim no)
-		(at 191.77 66.802 0)
+		(at 176.784 66.548 0)
 		(effects
 			(font
